File: schemat.brd (EAGLE design)
At the start: 160 x 100 mm, 43 parts, among them IC1 LM358N, Q1-1 IRFBG30, Q1-2 IRFBG30, Q1-3 IRFBG30, Q2-1 IRFBG30, Q2-2 IRFBG30, Q2-3 IRFBG30, Q3-1 IRFBG30, Q3-2 IRFBG30, Q3-3 IRFBG30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

Commit message: project finished
Parts:
- removed GND26: GND, con-faston:62221
- removed IC1: LM358N, linear:DIL08
- added GND_AUDIO, SECONDARY_GND: GND, con-faston:62221
- added IC2: LM321MF, linear:SOT23-5
- added U$1, U$10, U$11, U$12, U$2, U$3, U$4, U$5, U$6, U$7, U$8, U$9: (no value), heatsink:PF752
- moved Q4-3 281.1 mm to (143.6, 13.5), turned to 180 degrees
- moved C6 246.0 mm to (139.7, 29.5), flipped to the bottom, turned to 270 degrees
- moved Q4-2 234.9 mm to (119.6, 13.5), turned to 180 degrees
- moved AUDIO 224.0 mm to (6.35, 71.1)
- moved R8 212.7 mm to (14.9, 68.7), turned to 90 degrees
- moved PRIMARY_P1 204.7 mm to (152.4, 64.8)
- moved R7 198.2 mm to (35.6, 68.6), turned to 180 degrees
- moved PRIMARY_P2 197.1 mm to (152.4, 52.1)
- moved C8 195.0 mm to (38.2, 51.7), turned to 180 degrees
- moved C4 193.8 mm to (134.6, 30.7), turned to 270 degrees
- moved Q4-1 192.5 mm to (96.8, 13.5), turned to 180 degrees
- moved Q3-2 189.4 mm to (48.5, 13.5), turned to 180 degrees
- moved C9 187.8 mm to (27.9, 68.6), turned to 180 degrees
- moved C2 184.8 mm to (96.5, 30.5), turned to 270 degrees
- moved POT3 181.5 mm to (35.4, 48.1), turned to 270 degrees
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Connections:
- removed net N$12: GND26.1, R8.1
- removed net V+: IC1.8
- removed net V-: IC1.4
- removed net VCC: L1.1, POT3.1, R2.2, U2+U3.8, U4.1, U4.8
- new net 5V: C2.1, C3.1, IC2.5, POT3.1, R2.2, U1.3, U2+U3.8
- net 12V: now also L1.1; no longer C2.1, C3.1, U1.3
- net 12V_DRV: now also U4.1, U4.8
- net 12V_DRV1: now also IC2.1; no longer IC1.3
- net GND: now also GND_AUDIO.1, IC2.2, R8.1, SECONDARY_GND.1
- net N$10: now also IC2.3; no longer IC1.2
- net N$8: now also IC2.4; no longer IC1.1
Routing:
- net GND: track 0.00 -> 660.5 mm, vias 0 -> 26
- net PRIMARY_P2_Q: track 0.00 -> 428.5 mm
- net S1: track 0.00 -> 352.4 mm
- net 5V: track 0.00 -> 133.7 mm, vias 0 -> 4
- net 12V: track 0.00 -> 111.9 mm
- net 12V_DRV: track 0.00 -> 101.0 mm
- net N$1: track 0.00 -> 50.3 mm, vias 0 -> 1
- net N$8: track 0.00 -> 31.6 mm, vias 0 -> 2
- net N$2: track 0.00 -> 29.1 mm, vias 0 -> 1
- net N$4: track 0.00 -> 28.6 mm, vias 0 -> 3
- net N$5: track 0.00 -> 28.4 mm, vias 0 -> 1
- net N$11: track 0.00 -> 21.3 mm
- net 12V_DRV1: track 0.00 -> 16.4 mm, vias 0 -> 1
- net N$10: track 0.00 -> 14.8 mm, vias 0 -> 1
- net N$3: track 0.00 -> 7.32 mm
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Other:
- board text added: "12V"
- board text added: "AUDIO"

Commit message: transistor changed
Parts:
- removed PRIMARY_P1: V_SUPP, con-faston:62221
- removed Q1-1, Q1-2, Q1-3, Q2-1, Q2-2, Q2-3, Q3-1, Q3-2, Q3-3, Q4-1, Q4-2, Q4-3: IRFBG30, IRFBG30:TO220AB_VIS
- removed U$1, U$12, U$2, U$3, U$4, U$5, U$6, U$7: (no value), heatsink:PF752
- added Q1, Q2, Q3, Q4: SCT2450KEC, SCT2450KEC:TO545P521X1594X2583-3P
- moved U$8 25.4 mm to (116.8, 88.9)
- moved U$11 25.4 mm to (45.7, 88.9)
- moved U$10 25.4 mm to (69.8, 88.9)
- moved U$9 25.4 mm to (92.7, 88.9)
Connections:
- net GND: now also Q1.3, Q2.3, Q3.3, Q4.3; no longer Q1-1.2, Q1-2.2, Q1-3.2, Q2-1.2, Q2-2.2, Q2-3.2, Q3-1.2, Q3-2.2, Q3-3.2, Q4-1.2, Q4-2.2, Q4-3.2
- net PRIMARY_P2_Q: now also Q1.2, Q2.2, Q3.2, Q4.2; no longer Q1-1.3, Q1-2.3, Q1-3.3, Q2-1.3, Q2-2.3, Q2-3.3, Q3-1.3, Q3-2.3, Q3-3.3, Q4-1.3, Q4-2.3, Q4-3.3
- net S1: now also Q1.1, Q2.1, Q3.1, Q4.1; no longer Q1-1.1, Q1-2.1, Q1-3.1, Q2-1.1, Q2-2.1, Q2-3.1, Q3-1.1, Q3-2.1, Q3-3.1, Q4-1.1, Q4-2.1, Q4-3.1
Routing:
- net GND: track 660.5 -> 231.5 mm, vias 26 -> 4
- net PRIMARY_P2_Q: track 428.5 -> 0.00 mm
- net S1: track 352.4 -> 0.00 mm
